File: PCB/GPS_tracker_PCB.kicad_pcb (KiCad board)
At the start: 2 copper layers, 50 x 55.5 mm, 38 parts, among them CON1 Conn_ICSP, J1 Conn_Batt, J2 USB_A, J3 Conn_GPS, J4 Conn_GPS_LED, Q1 DMP1045U, SW1 SW_Reset, U1 MCP73831, U2 CP2102

Commit message: Current working version, most junk cleared out.
Parts:
- removed AC1: MMA8652FCR1, Housings_DFN_QFN:DFN-10_2x2mm_Pitch0.4mm
- removed C11, C12: 22 pF, Capacitors_SMD:C_1206
- removed Crystal1: 8MHz, Crystals:Crystal_HC49-4H_Vertical
- removed J4: Conn_GPS_LED, Pin_Headers:Pin_Header_Straight_1x01_Pitch1.00mm
- added ACCEL1: ADXL362, ADXL362:LGA-16_3.25x3.00, F.Cu at (104.2, 65.5)
- added C13: 10uF, Capacitors_SMD:C_1206, F.Cu at (105.2, 70.0)
- added C14: 0.1uF, Capacitors_SMD:C_1206, F.Cu at (105.2, 74.2)
- added C15: 0.1uF, Capacitors_SMD:C_1206, F.Cu at (111.0, 64.8)
- added R10: 10K, Resistors_SMD:R_1206, F.Cu at (140.6, 78.2)
- added R11: 10K, Resistors_SMD:R_1206, F.Cu at (135.2, 78.2)
- added R12: 10K, Resistors_SMD:R_1206, F.Cu at (126.2, 83.8)
- added R13: 10K, Resistors_SMD:R_1206, F.Cu at (130.8, 83.8)
- added R14: 10K, Resistors_SMD:R_1206, F.Cu at (135.2, 83.8)
- added R8: 10k, Resistors_SMD:R_1206, F.Cu at (113.5, 70.2)
- added R9: 10K, Resistors_SMD:R_1206, F.Cu at (129.8, 78.2)
- D1, D3, D4: footprint LEDs:LED_D5.0mm -> Diodes_SMD:D_0603
- VReg1: footprint TO_SOT_Packages_THT:TO-92_Molded_Wide_Oval -> TO_SOT_Packages_THT:TO-92_Inline_Wide
- moved R3 27.8 mm to (105.2, 78.8)
- moved C8 17.6 mm to (117.5, 64.8)
- moved R4 11.0 mm to (129.8, 73.2)
- moved C2 10.2 mm to (105.5, 103.2), turned to 0 degrees
- moved C6 5.62 mm to (111.2, 84.5)
- moved C3 5.35 mm to (105.2, 94.8), turned to 180 degrees
- moved C7 5.26 mm to (124.8, 64.8)
- moved R1 5.01 mm to (121.5, 82.8)
- moved C9 4.75 mm to (135.2, 73.2)
- moved C10 4.51 mm to (113.5, 77.0)
- moved R5 4.28 mm to (140.5, 73.2)
- moved C4 3.51 mm to (105.0, 83.2), turned to 0 degrees
- moved C5 3.50 mm to (105.0, 86.5)
- moved C1 2.02 mm to (116.0, 82.8)
Connections:
- MicroController1 pad 11: Net-(J4-Pad1) -> (no net)
- MicroController1 pad 12: /GPS_TX -> /GPS_RX
- MicroController1 pad 13: /GPS_RX -> /GPS_TX
- MicroController1 pad 2: (no net) -> /CS_ACC
- MicroController1 pad 23: (no net) -> /REC
- MicroController1 pad 27: /SDA -> (no net)
- MicroController1 pad 28: /SCL -> (no net)
- MicroController1 pad 32: /REC -> /INT_ACC
- MicroController1 pad 7: Net-(C12-Pad1) -> (no net)
- MicroController1 pad 8: Net-(C11-Pad1) -> (no net)
- SD1 pad 1: (no net) -> Net-(R11-Pad1)
- SD1 pad 8: (no net) -> Net-(R12-Pad1)
- Switch1 pad 9: (no net) -> VCC
Routing:
- net VCC: track 146.7 -> 190.5 mm, vias 1 -> 0
- net +5V: track 108.4 -> 151.8 mm, vias 0 -> 1
- net GND: track 249.5 -> 287.5 mm
- net /REC: track 70.4 -> 43.0 mm, vias 0 -> 1
- net Net-(C11-Pad1): track 27.3 -> 0.00 mm
- net Net-(C12-Pad1): track 25.4 -> 0.00 mm
- net /INT_ACC: track 0.00 -> 23.0 mm
- net /CS_ACC: track 0.00 -> 22.1 mm
- net Net-(J4-Pad1): track 17.5 -> 0.00 mm, vias 1 -> 0
- net /RESET: track 62.0 -> 47.4 mm, vias 2 -> 1
- net Net-(R11-Pad1): track 0.00 -> 11.9 mm
- net Net-(J2-Pad3): track 58.5 -> 47.3 mm, vias 0 -> 1
- net /CS_SD: track 27.8 -> 38.9 mm
- net /SDA: track 10.9 -> 0.00 mm, vias 2 -> 0
- net /SCL: track 10.5 -> 0.00 mm
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Other:
- board text added: "CLK"
- board text added: "GND"
- board text added: "MISO"
- board text added: "MOSI"
- board text added: "RST"
- board text added: "The Stopford GPS Tracker v1.1"
- board text added: "VCC"
- board text removed: "GPS Tracker v.1.0"
