File: PCB/GPS_tracker_PCB.sch (KiCad schematic (older format))
At the start: 38 parts, among them CON1 Conn_ICSP, J1 Conn_Batt, J2 USB_A, J3 Conn_GPS, J4 Conn_GPS_LED, Q1 DMP1045U, SW1 SW_Reset, U1 MCP73831, U2 CP2102

Commit message: Current working version, most junk cleared out.
Parts:
- removed AC1: MMA8652FCR1, Housings_DFN_QFN:DFN-10_2x2mm_Pitch0.4mm, symbol MMA8652FCR1
- removed C11, C12: 22 pF, Capacitors_SMD:C_1206, symbol C
- removed Crystal1: 8MHz, Crystals:Crystal_HC49-4H_Vertical, symbol Crystal
- removed J4: Conn_GPS_LED, Pin_Headers:Pin_Header_Straight_1x01_Pitch1.00mm, symbol Conn_01x01
- added ACCEL1: ADXL362, ADXL362:LGA-16_3.25x3.00, symbol ADXL362
- added C13: 10uF, Capacitors_SMD:C_1206, symbol C
- added C14, C15: 0.1uF, Capacitors_SMD:C_1206, symbol C
- added R10, R11, R12, R13, R14, R9: 10K, Resistors_SMD:R_1206, symbol R
- added R8: 10k, Resistors_SMD:R_1206, symbol R
- D1, D3, D4: footprint LEDs:LED_D5.0mm -> Diodes_SMD:D_0603
- J2: symbol USB_A -> USB_A-RESCUE-GPS_tracker_PCB
- VReg1: footprint TO_SOT_Packages_THT:TO-92_Molded_Wide_Oval -> TO_SOT_Packages_THT:TO-92_Inline_Wide
Connections:
- net labels added: CS_ACC, INT_ACC
- net labels removed: SCL, SDA
- wire segments 99 -> 129
- no-connect marks 31 -> 28
Other:
- note added: "SD card holder\nCHECK CONNECTIONS!"
- note added: "Too dim, change resistor"
- note removed: "SD card holder"
- moved on the sheet: CON1, J3, SD1
